Commit message: allow namespacing of xacro:include's
properties and macros in an included file will go into their own,
separate namespace, if the XML attribute `ns` is provided.
Access is by standard python syntax: namespace.name

File: test/include1.xacro (robot description, xacro)
@@ -1,4 +1,4 @@
 <a xmlns:xacro="http://www.ros.org/wiki/xacro">
 	<xacro:property name="var" value="1"/>
-	<xacro:macro name="foo1"><inc1/></xacro:macro>
+	<xacro:macro name="foo"><inc1/></xacro:macro>
 </a>

File: test/include2.xacro (robot description, xacro)
@@ -1,4 +1,4 @@
 <a xmlns:xacro="http://www.ros.org/wiki/xacro">
 	<xacro:property name="var" value="2"/>
-	<xacro:macro name="foo2"><inc2/></xacro:macro>
+	<xacro:macro name="foo"><inc2/></xacro:macro>
 </a>
